Commit message: feat: Added depth camera and LiDAR .xacro files for simulation

File: build/ors_robot/urdf/gazebo_control.xacro (robot description, xacro)
@@ -1 +1 @@
-/home/ebajit3/ors_ws/src/ors_robot/urdf/gazebo_control.xacro
+/home/ebajit/ors_ws/src/ors_robot/urdf/gazebo_control.xacro

File: build/ors_robot/urdf/robot.urdf.xacro (robot description, xacro)
@@ -1 +1 @@
-/home/ebajit3/ors_ws/src/ors_robot/urdf/robot.urdf.xacro
+/home/ebajit/ors_ws/src/ors_robot/urdf/robot.urdf.xacro

File: install/ors_robot/share/ors_robot/urdf/gazebo_control.xacro (robot description, xacro)
@@ -1 +1 @@
-/home/ebajit3/ors_ws/build/ors_robot/urdf/gazebo_control.xacro
+/home/ebajit/ors_ws/build/ors_robot/urdf/gazebo_control.xacro

File: install/ors_robot/share/ors_robot/urdf/robot.urdf.xacro (robot description, xacro)
@@ -1 +1 @@
-/home/ebajit3/ors_ws/build/ors_robot/urdf/robot.urdf.xacro
+/home/ebajit/ors_ws/build/ors_robot/urdf/robot.urdf.xacro

File: src/ors_robot/urdf/Robot_Base.urdf (robot description, URDF)
Before this commit: robot ors_robot, 7 links, 6 joints
Links:
- removed link M2M2_LIDAR
- removed link depth_cam
Joints:
- removed joint M2M2_LIDAR
- removed joint depth_cam

File: src/ors_robot/urdf/robot.urdf.xacro (robot description, xacro)
@@ -3,8 +3,7 @@
     <xacro:include filename="Robot_Base.urdf" />
     <xacro:include filename="gazebo_control.xacro"/>
-    <!-- <xacro:include filename="ros2_control.xacro"/>
-    <! <xacro:include filename="gazebo_control.xacro"/> -->
-    <!-- <xacro:include filename="lidar.xacro"/> -->
+    <xacro:include filename="depth_camera.xacro"/>
+    <xacro:include filename="lidar.xacro"/>
+    <!-- <xacro:include filename="ros2_control.xacro"/> -->
     <!-- <xacro:include filename="camera.xacro"/> -->
-    <!-- <xacro:include filename="depth_camera.xacro"/> -->
 </robot>
