Commit message: fix: meshes now display inside Gazebo and Rviz2. Modified rsp_sim.launch.py and Robot_Base.urdf to properly search for the .stl files for each component

File: src/ors_robot/urdf/Robot_Base.urdf (robot description, URDF)
Before this commit: robot ors_robot, 7 links, 6 joints
Links:
- link M2M2_LIDAR: geometry collision mesh filename=file://$(find ors_robot)/meshes/M2M2_LIDAR.STL; visual mesh filename=file://$(find ors_robot)/meshes/M2M2_LIDAR.STL
- link base_link: geometry collision mesh filename=file://$(find ors_robot)/meshes/base_link.STL; visual mesh filename=file://$(find ors_robot)/meshes/base_link.STL
- link depth_cam: geometry collision mesh filename=file://$(find ors_robot)/meshes/depth_cam.STL; visual mesh filename=file://$(find ors_robot)/meshes/depth_cam.STL
- link front_wheel: geometry collision mesh filename=file://$(find ors_robot)/meshes/front_wheel.STL; visual mesh filename=file://$(find ors_robot)/meshes/front_wheel.STL
- link left_wheel: geometry collision mesh filename=file://$(find ors_robot)/meshes/left_wheel.STL; visual mesh filename=file://$(find ors_robot)/meshes/left_wheel.STL
- link plate: geometry collision mesh filename=file://$(find ors_robot)/meshes/plate.STL; visual mesh filename=file://$(find ors_robot)/meshes/plate.STL
- link right_wheel: geometry collision mesh filename=file://$(find ors_robot)/meshes/right_wheel.STL; visual mesh filename=file://$(find ors_robot)/meshes/right_wheel.STL

Commit message: fix: Fixed wheel transform orientations which previously caused inverted movement when controlling robot with teleop_twist_keyboard

File: src/ors_robot/urdf/Robot_Base.urdf (robot description, URDF)
Before this commit: robot ors_robot, 7 links, 6 joints
Joints:
- removed joint front_wheel
- removed joint left_wheel
- removed joint right_wheel
- added joint front_wheel_joint: type continuous, parent base_link, child front_wheel, origin xyz=0.112773589774212 5.4823545785343E-05 0.00132877970694717 rpy=-1.5707963267949 0 0, axis 0 0 -1, limit effort=10 velocity=10
- added joint left_wheel_joint: type continuous, parent base_link, child left_wheel, origin xyz=-0.0129112176850158 -0.117664217504032 0.025328779706945 rpy=-1.5707963267949 1.5707963267949 0, axis 0 0 1, limit effort=10 velocity=10
- added joint right_wheel_joint: type continuous, parent base_link, child right_wheel, origin xyz=-0.0129112176873895 0.117549999993357 0.025328779706945 rpy=-1.5707963267949 1.5707963267949 0, axis 0 0 1, limit effort=10 velocity=10

File: src/ors_robot/urdf/gazebo_control.xacro (robot description, xacro)
@@ -4,7 +4,7 @@
         <plugin name="diff_drive" filename="libgazebo_ros_diff_drive.so">
             <!-- Wheel Information -->
-            <left_joint>left_wheel</left_joint>
-            <right_joint>right_wheel</right_joint>
-            <wheel_separation>7.03748170849394E−12</wheel_separation>
+            <left_joint>left_wheel_joint</left_joint>
+            <right_joint>right_wheel_joint</right_joint>
+            <wheel_separation>0.235</wheel_separation>
             <wheel_diameter>0.15</wheel_diameter>
             <!-- Limits -->

Commit message: feat: Implemented slam_toolbox, updated urdf and mesh files, added test.world as the default gazebo world when launching in sim mode

File: src/ors_robot/urdf/Robot_Base.urdf (robot description, URDF)
Before this commit: robot ors_robot, 5 links, 4 joints
Links:
- added link base_footprint
- link base_link: mass 3.75941738254691 -> 3.805
- link front_wheel: mass 0.00785398163397449 -> 0.007854
- link left_wheel: mass 0.0610725611857856 -> 0.061073
- link right_wheel: mass 0.0610725611857856 -> 0.061073
Joints:
- added joint base_footprint_joint: type fixed, parent base_link, child base_footprint, origin xyz=0 0 0 rpy=0 0 0
- joint front_wheel_joint: axis 0 0 -1 -> 0 1 0; origin xyz=0.112773589774212 5.4823545785343E-05 0.00132877970694717 rpy=-1.5707963267949 0 0 -> xyz=0.11327 5.4824E-05 0.0013288 rpy=0 0 0
- joint left_wheel_joint: origin xyz=-0.0129112176850158 -0.117664217504032 0.025328779706945 rpy=-1.5707963267949 1.5707963267949 0 -> xyz=-0.012911 0.11755 0.025329 rpy=-1.5707963267949 1.5707963267949 0
- joint plate: origin xyz=-0.0127165282933757 3.07436914599446E-05 0.239828779706945 rpy=0 0 0 -> xyz=-0.012717 3.0744E-05 0.23383 rpy=0 0 0
- joint right_wheel_joint: origin xyz=-0.0129112176873895 0.117549999993357 0.025328779706945 rpy=-1.5707963267949 1.5707963267949 0 -> xyz=-0.012911 -0.11766 0.025329 rpy=-1.5708 0 0

File: src/ors_robot/urdf/depth_camera.xacro (robot description, xacro)
@@ -5,15 +5,15 @@
     <inertial>
       <origin
-        xyz="-0.0131202485719072 -0.00185694854136453 -0.000475155115603476"
+        xyz="-0.01312 -0.0018569 -0.00047516"
         rpy="0 0 0" />
       <mass
-        value="0.118265203799494" />
+        value="0.11827" />
       <inertia
-        ixx="7.81722838749596E-05"
-        ixy="7.60380877739042E-07"
-        ixz="-3.98560089919681E-07"
-        iyy="9.42229928199424E-06"
-        iyz="-4.76491397960946E-09"
-        izz="7.76440264747213E-05" />
+        ixx="7.8172E-05"
+        ixy="7.6038E-07"
+        ixz="-3.9856E-07"
+        iyy="9.4223E-06"
+        iyz="-4.7652E-09"
+        izz="7.7644E-05" />
     </inertial>
     <visual>
@@ -28,5 +28,5 @@
         name="">
         <color
-          rgba="0.898039215686275 0.917647058823529 0.929411764705882 1" />
+          rgba="0.89804 0.91765 0.92941 1" />
       </material>
     </visual>
@@ -45,5 +45,5 @@
     type="fixed">
     <origin
-      xyz="0.149440914994276 0.00218526482966985 0.0123528880010465"
+      xyz="0.14944 0.0021853 0.012353"
       rpy="0 0 0" />
     <parent

File: src/ors_robot/urdf/gazebo_control.xacro (robot description, xacro)
@@ -4,6 +4,6 @@
         <plugin name="diff_drive" filename="libgazebo_ros_diff_drive.so">
             <!-- Wheel Information -->
-            <left_joint>right_wheel_joint</left_joint>
-            <right_joint>left_wheel_joint</right_joint>
+            <left_joint>left_wheel_joint</left_joint>
+            <right_joint>right_wheel_joint</right_joint>
             <wheel_separation>0.23521</wheel_separation>
             <wheel_diameter>0.15</wheel_diameter>

File: src/ors_robot/urdf/lidar.xacro (robot description, xacro)
@@ -3,7 +3,7 @@
   <link name="M2M2_LIDAR">
     <inertial>
-      <origin xyz="0.000544180788152326 -0.000121760206787558 -0.0676836000482276" rpy="0 0 0" />
-      <mass value="0.144547687439008" />
-      <inertia ixx="0.000167357888369665" ixy="7.58898386397937E-10" ixz="1.54108302065642E-08" iyy="0.000166948275602806" iyz="4.60881838904236E-08" izz="0.000189951798778922" />
+      <origin xyz="-0.0011981 -0.0001963 -0.067684" rpy="0 0 0" />
+      <mass value="0.14455" />
+      <inertia ixx="0.00016736" ixy="3.546E-08" ixz="1.4853E-08" iyy="0.00016695" iyz="4.7103E-08" izz="0.00018995" />
     </inertial>
     <visual>
@@ -13,5 +13,5 @@
       </geometry>
       <material name="">
-        <color rgba="0.792156862745098 0.819607843137255 0.933333333333333 1" />
+        <color rgba="0.79216 0.81961 0.93333 1" />
       </material>
     </visual>
@@ -24,5 +24,5 @@
   </link>
   <joint name="M2M2_LIDAR" type="fixed">
-    <origin xyz="0.011257243470593 -5.35218498943779E-05 0.1054" rpy="0 0 0" />
+    <origin xyz="0.0016059 4.6046E-05 0.1054" rpy="0 0 0" />
     <parent link="plate" />
     <child link="M2M2_LIDAR" />
@@ -33,5 +33,5 @@
         <sensor name="laser" type="ray">
             <pose> 0 0 0 0 0 0 </pose>
-            <visualize>true</visualize>
+            <visualize>false</visualize>
             <update_rate>10</update_rate>
             <ray>
@@ -45,5 +45,5 @@
                 <range>
                     <min>0.3</min>
-                    <max>12</max>
+                    <max>20</max>
                 </range>
             </ray>
