Commit message: fix: update urdf for SLAM standards

File: src/ors_robot/urdf/robot.urdf.xacro (robot description, xacro)
@@ -1,5 +1,5 @@
 <?xml version="1.0"?>
 <robot xmlns:xacro="http://www.ros.org/wiki/xacro"  name="robot">
-    <xacro:include filename="Robot_Base.urdf" />
+    <xacro:include filename="robot_core.urdf" />
     <xacro:include filename="gazebo_control.xacro"/>
     <xacro:include filename="depth_camera.xacro"/>

File: src/ors_robot/urdf/robot_core.urdf (robot description, URDF)
Before this commit: robot ors_robot, 6 links, 5 joints
Links:
- added link chassis, mass 3.805; collision mesh filename=file://$(find ors_robot)/meshes/base_link.STL; visual mesh filename=file://$(find ors_robot)/meshes/base_link.STL
- link base_link: mass 3.805 -> None; geometry 
Joints:
- added joint chassis_joint: type fixed, parent base_link, child chassis, origin xyz=0 0 0.042377
