Commit message: refactor: Format urdf

File: src/ors_robot/urdf/lidar.xacro (robot description, xacro)
@@ -1,56 +1,31 @@
 <?xml version="1.0"?>
 <robot xmlns:xacro="http://www.ros.org/wiki/xacro" >
-  <link
-    name="M2M2_LIDAR">
+  <link name="M2M2_LIDAR">
     <inertial>
-      <origin
-        xyz="0.000544180788152326 -0.000121760206787558 -0.0676836000482276"
-        rpy="0 0 0" />
-      <mass
-        value="0.144547687439008" />
-      <inertia
-        ixx="0.000167357888369665"
-        ixy="7.58898386397937E-10"
-        ixz="1.54108302065642E-08"
-        iyy="0.000166948275602806"
-        iyz="4.60881838904236E-08"
-        izz="0.000189951798778922" />
+      <origin xyz="0.000544180788152326 -0.000121760206787558 -0.0676836000482276" rpy="0 0 0" />
+      <mass value="0.144547687439008" />
+      <inertia ixx="0.000167357888369665" ixy="7.58898386397937E-10" ixz="1.54108302065642E-08" iyy="0.000166948275602806" iyz="4.60881838904236E-08" izz="0.000189951798778922" />
     </inertial>
     <visual>
-      <origin
-        xyz="0 0 0"
-        rpy="0 0 0" />
+      <origin xyz="0 0 0" rpy="0 0 0" />
       <geometry>
-        <mesh
-          filename="file://$(find ors_robot)/meshes/M2M2_LIDAR.STL" />
+        <mesh filename="file://$(find ors_robot)/meshes/M2M2_LIDAR.STL" />
       </geometry>
-      <material
-        name="">
-        <color
-          rgba="0.792156862745098 0.819607843137255 0.933333333333333 1" />
+      <material name="">
+        <color rgba="0.792156862745098 0.819607843137255 0.933333333333333 1" />
       </material>
     </visual>
     <collision>
-      <origin
-        xyz="0 0 0"
-        rpy="0 0 0" />
+      <origin xyz="0 0 0" rpy="0 0 0" />
       <geometry>
-        <mesh
-          filename="file://$(find ors_robot)/meshes/M2M2_LIDAR.STL" />
+        <mesh filename="file://$(find ors_robot)/meshes/M2M2_LIDAR.STL" />
       </geometry>
     </collision>
   </link>
-  <joint
-    name="M2M2_LIDAR"
-    type="fixed">
-    <origin
-      xyz="0.011257243470593 -5.35218498943779E-05 0.1054"
-      rpy="0 0 0" />
-    <parent
-      link="plate" />
-    <child
-      link="M2M2_LIDAR" />
-    <axis
-      xyz="0 0 0" />
+  <joint name="M2M2_LIDAR" type="fixed">
+    <origin xyz="0.011257243470593 -5.35218498943779E-05 0.1054" rpy="0 0 0" />
+    <parent link="plate" />
+    <child link="M2M2_LIDAR" />
+    <axis xyz="0 0 0" />
   </joint>
     <gazebo reference="M2M2_LIDAR">

Commit message: fix: replace m2m2 with rplidar

File: src/ors_robot/urdf/lidar.xacro (robot description, xacro)
@@ -1,38 +1,39 @@
 <?xml version="1.0"?>
-<robot xmlns:xacro="http://www.ros.org/wiki/xacro" >
-  <link name="M2M2_LIDAR">
-    <inertial>
-      <origin xyz="-0.0011981 -0.0001963 -0.067684" rpy="0 0 0" />
-      <mass value="0.14455" />
-      <inertia ixx="0.00016736" ixy="3.546E-08" ixz="1.4853E-08" iyy="0.00016695" iyz="4.7103E-08" izz="0.00018995" />
-    </inertial>
-    <visual>
-      <origin xyz="0 0 0" rpy="0 0 0" />
-      <geometry>
-        <mesh filename="file://$(find ors_robot)/meshes/M2M2_LIDAR.STL" />
-      </geometry>
-      <material name="">
-        <color rgba="0.79216 0.81961 0.93333 1" />
-      </material>
-    </visual>
-    <collision>
-      <origin xyz="0 0 0" rpy="0 0 0" />
-      <geometry>
-        <mesh filename="file://$(find ors_robot)/meshes/M2M2_LIDAR.STL" />
-      </geometry>
-    </collision>
-  </link>
-  <joint name="M2M2_LIDAR" type="fixed">
-    <origin xyz="0.0016059 4.6046E-05 0.1054" rpy="0 0 0" />
-    <parent link="plate" />
-    <child link="M2M2_LIDAR" />
-    <axis xyz="0 0 0" />
-  </joint>
-    <gazebo reference="M2M2_LIDAR">
+<robot xmlns:xacro="http://www.ros.org/wiki/xacro"  name="robot">
+    <!-- Add a joint and link to locate LiDar within our robot -->
+    <joint name="laser_joint" type="fixed">
+        <parent link="chassis"/>
+        <child link="laser_frame"/>
+        <!-- Place origin of laser link at the top of the robot -->
+        <origin xyz="0.1 0 0.175" rpy="0 0 0"/>
+    </joint>
+    <link name="laser_frame">
+        <visual>
+            <geometry>
+                <cylinder radius="0.05" length="0.05"/>
+            </geometry>
+            <material name="red"/>
+        </visual>
+        <collision>
+            <geometry>
+                <cylinder radius="0.05" length="0.05"/>
+            </geometry>
+        </collision>
+        <xacro:inertial_cylinder mass="0.1" length="0.4" radius="0.05">
+            <origin xyz="0 0 0" rpy="0 0 0"/>
+        </xacro:inertial_cylinder>
+    </link>
+    <!-- Add a gazebo tag to simulate the LiDar -->
+    <gazebo reference="laser_frame">
+        <!-- Set the color of the LiDar. The color for the link sets color in rviz, not Gazebo -->
         <material>Gazebo/Red</material>
+        <!-- Ray sensor is a scanning LiDar -->
         <sensor name="laser" type="ray">
+            <!-- Origin of the sensor is at the center of the link -->
             <pose> 0 0 0 0 0 0 </pose>
             <visualize>false</visualize>
+            <!-- Update 10 times / second -->
             <update_rate>10</update_rate>
+            <!-- Specify paramters for the virtual sensor -->
             <ray>
                 <scan>
@@ -45,13 +46,16 @@
                 <range>
                     <min>0.3</min>
-                    <max>20</max>
+                    <max>12</max>
                 </range>
             </ray>
+            <!-- Plug in to publish the gazebo ray sensor to ROS topics -->
             <plugin name="laser_controller" filename="libgazebo_ros_ray_sensor.so">
+                <!-- What topic to publish onto (publish to scan) -->
                 <ros>
-                    <argument>--ros-args --remap ~/out:=scan</argument>
+                    <argument>~/out:=scan</argument>
                 </ros>
                 <output_type>sensor_msgs/LaserScan</output_type>
-                <frame_name>M2M2_LIDAR</frame_name>
+                <!-- What frame ID to put in the laser scan message -->
+                <frame_name>laser_frame</frame_name>
             </plugin>
         </sensor>

Commit message: fix: lidar xacro

File: src/ors_robot/urdf/lidar.xacro (robot description, xacro)
@@ -1,7 +1,11 @@
 <?xml version="1.0"?>
 <robot xmlns:xacro="http://www.ros.org/wiki/xacro"  name="robot">
+    <!-- Define material 'red' -->
+    <material name="red">
+        <color rgba="1 0 0 1"/>
+    </material>
     <!-- Add a joint and link to locate LiDar within our robot -->
     <joint name="laser_joint" type="fixed">
-        <parent link="chassis"/>
+        <parent link="plate"/>
         <child link="laser_frame"/>
         <!-- Place origin of laser link at the top of the robot -->
@@ -20,7 +24,15 @@
             </geometry>
         </collision>
-        <xacro:inertial_cylinder mass="0.1" length="0.4" radius="0.05">
-            <origin xyz="0 0 0" rpy="0 0 0"/>
-        </xacro:inertial_cylinder>
+      <inertial>
+          <mass value="0.1"/>
+          <inertia
+              ixx="0.000016"
+              ixy="0"
+              ixz="0"
+              iyy="0.000016"
+              iyz="0"
+              izz="0.000025"/>
+          <origin xyz="0 0 0" rpy="0 0 0"/>
+      </inertial>
     </link>
     <!-- Add a gazebo tag to simulate the LiDar -->

Commit message: fix: plate joint

File: src/ors_robot/urdf/lidar.xacro (robot description, xacro)
@@ -24,15 +24,15 @@
             </geometry>
         </collision>
-      <inertial>
-          <mass value="0.1"/>
-          <inertia
-              ixx="0.000016"
-              ixy="0"
-              ixz="0"
-              iyy="0.000016"
-              iyz="0"
-              izz="0.000025"/>
-          <origin xyz="0 0 0" rpy="0 0 0"/>
-      </inertial>
+        <inertial>
+            <mass value="0.1"/>
+            <inertia
+                ixx="0.000016"
+                ixy="0"
+                ixz="0"
+                iyy="0.000016"
+                iyz="0"
+                izz="0.000025"/>
+            <origin xyz="0 0 0" rpy="0 0 0"/>
+        </inertial>
     </link>
     <!-- Add a gazebo tag to simulate the LiDar -->

File: src/ors_robot/urdf/robot_core.urdf (robot description, URDF)
Before this commit: robot ors_robot, 7 links, 6 joints
Joints:
- removed joint plate
- added joint plate_joint: type fixed, parent base_link, child plate, origin xyz=-0.012717 3.0744E-05 0.23383 rpy=0 0 0, axis 0 0 0

Commit message: fix?: publish laser_frame from base_link

File: src/ors_robot/urdf/lidar.xacro (robot description, xacro)
@@ -7,5 +7,5 @@
     <!-- Add a joint and link to locate LiDar within our robot -->
     <joint name="laser_joint" type="fixed">
-        <parent link="plate"/>
+        <parent link="base_link"/>
         <child link="laser_frame"/>
         <!-- Place origin of laser link at the top of the robot -->
