Commit message: fix?: Remove static publishing of base_link and base_footprint, create 3 publishes this

File: src/ors_robot/urdf/robot_core.urdf (robot description, URDF)
Before this commit: robot ors_robot, 7 links, 6 joints
Links:
- removed link base_footprint
- removed link base_link
Joints:
- removed joint base_footprint_joint
