Commit message: fix?: ignore lidar xacro and directly publish tf from stl271.launch.py

File: src/ors_robot/urdf/depth_camera.xacro (robot description, xacro)
@@ -46,11 +46,9 @@
     <origin
       xyz="0.14944 0.0021853 0.012353"
-      rpy="0 0 0" />
-    <parent
-      link="plate" />
-    <child
-      link="depth_cam_link" />
-    <axis
-      xyz="0 0 0" />
+      rpy="0 0 0"
+    />
+    <parent link="plate" />
+    <child link="depth_cam_link" />
+    <axis xyz="0 0 0" />
   </joint>
     <joint name="depth_cam_optical_joint" type="fixed">

File: src/ors_robot/urdf/lidar.xacro (robot description, xacro)
@@ -7,5 +7,5 @@
     <!-- Add a joint and link to locate LiDar within our robot -->
     <joint name="laser_joint" type="fixed">
-        <parent link="base_link"/>
+        <parent link="plate"/>
         <child link="laser_frame"/>
         <!-- Place origin of laser link at the top of the robot -->
@@ -36,16 +36,11 @@
         </inertial>
     </link>
-    <!-- Add a gazebo tag to simulate the LiDar -->
+    <!--
     <gazebo reference="laser_frame">
-        <!-- Set the color of the LiDar. The color for the link sets color in rviz, not Gazebo -->
         <material>Gazebo/Red</material>
-        <!-- Ray sensor is a scanning LiDar -->
         <sensor name="laser" type="ray">
-            <!-- Origin of the sensor is at the center of the link -->
             <pose> 0 0 0 0 0 0 </pose>
             <visualize>false</visualize>
-            <!-- Update 10 times / second -->
             <update_rate>10</update_rate>
-            <!-- Specify paramters for the virtual sensor -->
             <ray>
                 <scan>
@@ -61,15 +56,12 @@
                 </range>
             </ray>
-            <!-- Plug in to publish the gazebo ray sensor to ROS topics -->
             <plugin name="laser_controller" filename="libgazebo_ros_ray_sensor.so">
-                <!-- What topic to publish onto (publish to scan) -->
                 <ros>
                     <argument>~/out:=scan</argument>
                 </ros>
                 <output_type>sensor_msgs/LaserScan</output_type>
-                <!-- What frame ID to put in the laser scan message -->
                 <frame_name>laser_frame</frame_name>
             </plugin>
         </sensor>
-    </gazebo>
+    </gazebo> -->
 </robot>

File: src/ors_robot/urdf/robot.urdf.xacro (robot description, xacro)
@@ -4,5 +4,5 @@
     <xacro:include filename="gazebo_control.xacro"/>
     <xacro:include filename="depth_camera.xacro"/>
-    <xacro:include filename="lidar.xacro"/>
+    <!-- <xacro:include filename="lidar.xacro"/> -->
     <!-- <xacro:include filename="ros2_control.xacro"/> -->
     <!-- <xacro:include filename="camera.xacro"/> -->

Commit message: fix: lidar and depth urdf

File: src/ors_robot/urdf/depth_camera.xacro (robot description, xacro)
@@ -79,5 +79,5 @@
             <plugin name="camera_controller" filename="libgazebo_ros_camera.so">
                 <frame_name>depth_cam_link_optical</frame_name>
-                <min_depth>0.1</min_depth>
+                <min_depth>0.2</min_depth>
                 <max_depth>100.0</max_depth>
             </plugin>

File: src/ors_robot/urdf/lidar.xacro (robot description, xacro)
@@ -1,7 +1,7 @@
 <?xml version="1.0"?>
 <robot xmlns:xacro="http://www.ros.org/wiki/xacro"  name="robot">
-    <!-- Define material 'red' -->
-    <material name="red">
-        <color rgba="1 0 0 1"/>
+    <!-- Define material 'grey' -->
+    <material name="grey">
+        <color rgba="0.7 0.7 0.7 1"/>
     </material>
     <!-- Add a joint and link to locate LiDar within our robot -->
@@ -10,5 +10,5 @@
         <child link="laser_frame"/>
         <!-- Place origin of laser link at the top of the robot -->
-        <origin xyz="0.1 0 0.175" rpy="0 0 0"/>
+        <origin xyz="0 0 0.06" rpy="0 0 0"/>
     </joint>
     <link name="laser_frame">

File: src/ors_robot/urdf/robot_core.urdf (robot description, URDF)
Before this commit: robot ors_robot, 7 links, 6 joints
Joints:
- joint plate: origin xyz=-0.012717 3.0744E-05 0.23383 rpy=0 0 0 -> xyz=-0.012717 3.0744E-05 0.27492297775729 rpy=0 0 0
